File: 1-ECAD/cyberman/Project Architecture.kicad_sch (KiCad schematic)
At the start: 0 parts

Commit message: power page close
siuuuuuuuuuuuu
Other:
- sheet MCU - IOs ports: added DSP{CS RST TP_INT}, FG_ALRT, I2C_AUX{SCL SDA}, I2C_BOARD{SCL SDA}, I2S{SCK SD WS}, IMU{INT1 INT2}, MAG.INT, PWR{INT RST PERIPH}, SPK.SD; removed BOARD_I2C{SCL SDA}, DSP{CS RST}
- sheet Power ports: added FG_ALRT, PWR{INT RST PERIPH}; removed PWR{PERIPH RST}
- note added: "Page 7"
- note added: "Page 8"
- note added: "Page 9"
