File: 1-ECAD/cyberman/Revision History.kicad_sch (KiCad schematic)
At the start: 0 parts

Commit message: new changes
close display page and peripheral schematic
Other:
- company: ${COMPANY} -> kode.
Changed lines of the file:
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@@
 	(title_block
 		(title "Revision History")
-		(date "Last Modified Date")
-		(rev "${REVISION}")
-		(company "${COMPANY}")
+		(date "2024-12-11")
+		(rev "1.0")
+		(company "kode.")
 	)
 	(polyline
