File: 1-ECAD/cyberman/peripherals.kicad_sch (KiCad schematic)
At the start: 88 parts, among them J801 5033981892, J802 Conn_01x04, SW801 SKRMAAE010, SW802 SKRMAAE010, SW803 SKRMAAE010, SW804 SKRMAAE010, SW805 SKRMAAE010, SW806 SKRMAAE010, U801 PM254-2-10-W-8.5

Commit message: power page close
siuuuuuuuuuuuu
Changed lines of the file:
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@@
 	(title_block
 		(title "Peripherals")
-		(date "2024-12-11")
+		(date "2024-12-18")
 		(rev "1.0")
 		(company "kode.")
@@
 	)
 	(bus_entry
+		(at 114.3 243.84)
+		(size -2.54 2.54)
+		(stroke
+			(width 0)
+			(type default)
+		)
+	)
+	(bus_entry
 		(at 50.8 243.84)
 		(size -2.54 2.54)
@@
 	)
 	(bus_entry
+		(at 114.3 246.38)
+		(size -2.54 2.54)
+		(stroke
+			(width 0)
+			(type default)
+		)
+	)
+	(bus_entry
 		(at 50.8 248.92)
 		(size -2.54 2.54)
@@
 	(wire
 		(pts
+			(xy 96.52 246.38) (xy 111.76 246.38)
+		)
+		(stroke
+			(width 0)
+			(type default)
+		)
+	)
+	(wire
+		(pts
 			(xy 356.87 77.47) (xy 356.87 85.09)
 		)
@@
 		)
 	)
+	(bus
+		(pts
+			(xy 114.3 243.84) (xy 114.3 246.38)
+		)
+		(stroke
+			(width 0)
+			(type default)
+		)
+	)
 	(wire
 		(pts
@@
 	(wire
 		(pts
+			(xy 96.52 248.92) (xy 111.76 248.92)
+		)
+		(stroke
+			(width 0)
+			(type default)
+		)
+	)
+	(wire
+		(pts
 			(xy 254 177.8) (xy 269.24 177.8)
 		)
@@
 		)
 	)
+	(bus
+		(pts
+			(xy 114.3 241.3) (xy 114.3 243.84)
+		)
+		(stroke
+			(width 0)
+			(type default)
+		)
+	)
 	(wire
 		(pts
@@
 		)
 	)
+	(text_box "DESIGN NOTE:\nLED"
+		(exclude_from_sim no)
+		(at 168.91 236.22 0)
+		(size 30.48 20.32)
+		(stroke
+			(width 1.5)
+			(type solid)
+			(color 255 0 0 1)
+		)
+		(fill
+			(type none)
+		)
+		(effects
+			(font
+				(face "Times New Roman")
+				(size 2 2)
+				(thickness 0.4)
+				(bold yes)
+				(color 255 0 0 1)
+			)
+			(justify left top)
+		)
+	)
 	(text "microSD Connector"
 		(exclude_from_sim no)
@@
 		)
 	)
+	(label "I2C_BOARD.SCL"
+		(at 96.52 246.38 0)
+		(fields_autoplaced yes)
+		(effects
+			(font
+				(size 1.27 1.27)
+			)
+			(justify left bottom)
+		)
+	)
 	(label "BUTTON.TOP"
 		(at 33.02 248.92 0)
@@
 		)
 	)
+	(label "I2C_BOARD.SDA"
+		(at 96.52 248.92 0)
+		(fields_autoplaced yes)
+		(effects
+			(font
+				(size 1.27 1.27)
+			)
+			(justify left bottom)
+		)
+	)
 	(label "SD.CLK"
 		(at 250.19 67.31 0)
@@
 		)
 	)
+	(hierarchical_label "I2C_BOARD{SCL SDA}"
+		(shape input)
+		(at 114.3 241.3 0)
+		(fields_autoplaced yes)
+		(effects
+			(font
+				(size 1.27 1.27)
+			)
+			(justify left)
+		)
+	)
 	(symbol
 		(lib_id "0_resistor_smd:RC0402FR-07330RL")
@@
 		(dnp no)
 		(fields_autoplaced yes)
-		(property "Reference" "#PWR0802"
+		(property "Reference" "#PWR802"
 			(at 106.68 48.26 0)
 			(effects
@@
 			(project ""
 				(path "/0650c7a8-acba-429c-9f8e-eec0baf0bc1c/fede4c36-00cc-4d3d-b71c-5243ba232202/7c79e64d-6bcf-40af-a5ad-7c52beef15e9"
-					(reference "#PWR0802")
+					(reference "#PWR802")
 					(unit 1)
 				)
@@
 		(dnp no)
 		(fields_autoplaced yes)
-		(property "Reference" "#PWR0811"
+		(property "Reference" "#PWR811"
 			(at 91.44 173.99 0)
 			(effects
@@
 			(project "cyberman"
 				(path "/0650c7a8-acba-429c-9f8e-eec0baf0bc1c/fede4c36-00cc-4d3d-b71c-5243ba232202/7c79e64d-6bcf-40af-a5ad-7c52beef15e9"
-					(reference "#PWR0811")
+					(reference "#PWR811")
 					(unit 1)
 				)
@@
 		(dnp no)
 		(fields_autoplaced yes)
-		(property "Reference" "#PWR0807"
+		(property "Reference" "#PWR807"
 			(at 287.02 151.13 0)
 			(effects
@@
 			(project "cyberman"
 				(path "/0650c7a8-acba-429c-9f8e-eec0baf0bc1c/fede4c36-00cc-4d3d-b71c-5243ba232202/7c79e64d-6bcf-40af-a5ad-7c52beef15e9"
-					(reference "#PWR0807")
+					(reference "#PWR807")
 					(unit 1)
 				)
@@
 		(dnp no)
 		(fields_autoplaced yes)
-		(property "Reference" "#PWR0808"
+		(property "Reference" "#PWR808"
 			(at 322.58 151.13 0)
 			(effects
@@
 			(project "cyberman"
 				(path "/0650c7a8-acba-429c-9f8e-eec0baf0bc1c/fede4c36-00cc-4d3d-b71c-5243ba232202/7c79e64d-6bcf-40af-a5ad-7c52beef15e9"
-					(reference "#PWR0808")
+					(reference "#PWR808")
 					(unit 1)
 				)
@@
 		(dnp no)
 		(fields_autoplaced yes)
-		(property "Reference" "#PWR0804"
+		(property "Reference" "#PWR804"
 			(at 356.87 101.6 0)
 			(effects
@@
 			(project ""
 				(path "/0650c7a8-acba-429c-9f8e-eec0baf0bc1c/fede4c36-00cc-4d3d-b71c-5243ba232202/7c79e64d-6bcf-40af-a5ad-7c52beef15e9"
-					(reference "#PWR0804")
+					(reference "#PWR804")
 					(unit 1)
 				)
@@
 		(dnp no)
 		(fields_autoplaced yes)
-		(property "Reference" "#PWR0814"
+		(property "Reference" "#PWR814"
 			(at 322.58 194.31 0)
 			(effects
@@
 			(project "cyberman"
 				(path "/0650c7a8-acba-429c-9f8e-eec0baf0bc1c/fede4c36-00cc-4d3d-b71c-5243ba232202/7c79e64d-6bcf-40af-a5ad-7c52beef15e9"
-					(reference "#PWR0814")
+					(reference "#PWR814")
 					(unit 1)
 				)
@@
 		(dnp no)
 		(fields_autoplaced yes)
-		(property "Reference" "#PWR0810"
+		(property "Reference" "#PWR810"
 			(at 340.36 158.75 0)
 			(effects
@@
 			(project "cyberman"
 				(path "/0650c7a8-acba-429c-9f8e-eec0baf0bc1c/fede4c36-00cc-4d3d-b71c-5243ba232202/7c79e64d-6bcf-40af-a5ad-7c52beef15e9"
-					(reference "#PWR0810")
+					(reference "#PWR810")
 					(unit 1)
 				)
@@
 		(dnp no)
 		(fields_autoplaced yes)
-		(property "Reference" "#PWR0806"
+		(property "Reference" "#PWR806"
 			(at 170.18 137.16 0)
 			(effects
@@
 			(project ""
 				(path "/0650c7a8-acba-429c-9f8e-eec0baf0bc1c/fede4c36-00cc-4d3d-b71c-5243ba232202/7c79e64d-6bcf-40af-a5ad-7c52beef15e9"
-					(reference "#PWR0806")
+					(reference "#PWR806")
 					(unit 1)
 				)
@@
 		(dnp no)
 		(fields_autoplaced yes)
-		(property "Reference" "#PWR0812"
+		(property "Reference" "#PWR812"
 			(at 73.66 181.61 0)
 			(effects
@@
 			(project "cyberman"
 				(path "/0650c7a8-acba-429c-9f8e-eec0baf0bc1c/fede4c36-00cc-4d3d-b71c-5243ba232202/7c79e64d-6bcf-40af-a5ad-7c52beef15e9"
-					(reference "#PWR0812")
+					(reference "#PWR812")
 					(unit 1)
 				)
@@
 		(dnp no)
 		(fields_autoplaced yes)
-		(property "Reference" "#PWR0815"
+		(property "Reference" "#PWR815"
 			(at 121.92 201.93 0)
 			(effects
@@
 			(project "cyberman"
 				(path "/0650c7a8-acba-429c-9f8e-eec0baf0bc1c/fede4c36-00cc-4d3d-b71c-5243ba232202/7c79e64d-6bcf-40af-a5ad-7c52beef15e9"
-					(reference "#PWR0815")
+					(reference "#PWR815")
 					(unit 1)
 				)
@@
 		(dnp no)
 		(fields_autoplaced yes)
-		(property "Reference" "#PWR0813"
+		(property "Reference" "#PWR813"
 			(at 287.02 194.31 0)
 			(effects
@@
 			(project ""
 				(path "/0650c7a8-acba-429c-9f8e-eec0baf0bc1c/fede4c36-00cc-4d3d-b71c-5243ba232202/7c79e64d-6bcf-40af-a5ad-7c52beef15e9"
-					(reference "#PWR0813")
+					(reference "#PWR813")
 					(unit 1)
 				)
@@
 		(dnp no)
 		(fields_autoplaced yes)
-		(property "Reference" "#PWR0809"
+		(property "Reference" "#PWR809"
 			(at 270.51 158.75 0)
 			(effects
@@
 			(project "cyberman"
 				(path "/0650c7a8-acba-429c-9f8e-eec0baf0bc1c/fede4c36-00cc-4d3d-b71c-5243ba232202/7c79e64d-6bcf-40af-a5ad-7c52beef15e9"
-					(reference "#PWR0809")
+					(reference "#PWR809")
 					(unit 1)
 				)
@@
 		(dnp no)
 		(fields_autoplaced yes)
-		(property "Reference" "#PWR0805"
+		(property "Reference" "#PWR805"
 			(at 290.83 111.76 0)
 			(effects
@@
 			(project "cyberman"
 				(path "/0650c7a8-acba-429c-9f8e-eec0baf0bc1c/fede4c36-00cc-4d3d-b71c-5243ba232202/7c79e64d-6bcf-40af-a5ad-7c52beef15e9"
-					(reference "#PWR0805")
+					(reference "#PWR805")
 					(unit 1)
 				)
@@
 		(dnp no)
 		(fields_autoplaced yes)
-		(property "Reference" "#PWR0803"
+		(property "Reference" "#PWR803"
 			(at 241.3 66.04 0)
 			(effects
@@
 			(project "cyberman"
 				(path "/0650c7a8-acba-429c-9f8e-eec0baf0bc1c/fede4c36-00cc-4d3d-b71c-5243ba232202/7c79e64d-6bcf-40af-a5ad-7c52beef15e9"
-					(reference "#PWR0803")
+					(reference "#PWR803")
 					(unit 1)
 				)
@@
 		(dnp no)
 		(fields_autoplaced yes)
-		(property "Reference" "#PWR0801"
+		(property "Reference" "#PWR801"
 			(at 241.3 46.99 0)
 			(effects
@@
 			(project "cyberman"
 				(path "/0650c7a8-acba-429c-9f8e-eec0baf0bc1c/fede4c36-00cc-4d3d-b71c-5243ba232202/7c79e64d-6bcf-40af-a5ad-7c52beef15e9"
-					(reference "#PWR0801")
+					(reference "#PWR801")
 					(unit 1)
 				)
@@
 		(dnp no)
 		(fields_autoplaced yes)
-		(property "Reference" "#PWR0817"
+		(property "Reference" "#PWR817"
 			(at 363.22 212.09 0)
 			(effects
@@
 			(project "cyberman"
 				(path "/0650c7a8-acba-429c-9f8e-eec0baf0bc1c/fede4c36-00cc-4d3d-b71c-5243ba232202/7c79e64d-6bcf-40af-a5ad-7c52beef15e9"
-					(reference "#PWR0817")
+					(reference "#PWR817")
 					(unit 1)
 				)
@@
 		(dnp no)
 		(fields_autoplaced yes)
-		(property "Reference" "#PWR0818"
+		(property "Reference" "#PWR818"
 			(at 66.04 217.17 0)
 			(effects
@@
 			(project "cyberman"
 				(path "/0650c7a8-acba-429c-9f8e-eec0baf0bc1c/fede4c36-00cc-4d3d-b71c-5243ba232202/7c79e64d-6bcf-40af-a5ad-7c52beef15e9"
-					(reference "#PWR0818")
+					(reference "#PWR818")
 					(unit 1)
 				)
@@
 		(dnp no)
 		(fields_autoplaced yes)
-		(property "Reference" "#PWR0816"
+		(property "Reference" "#PWR816"
 			(at 246.38 212.09 0)
 			(effects
@@
 			(project "cyberman"
 				(path "/0650c7a8-acba-429c-9f8e-eec0baf0bc1c/fede4c36-00cc-4d3d-b71c-5243ba232202/7c79e64d-6bcf-40af-a5ad-7c52beef15e9"
-					(reference "#PWR0816")
+					(reference "#PWR816")
 					(unit 1)
 				)
