File: 1-ECAD/cyberman/sensors-audio.kicad_sch (KiCad schematic)
At the start: 19 parts, among them J1001 532610271, U1001 MAX98357A, U1002 ICS-43434, U1003 LIS2MDLTR, U1004 LSM6DSOTR

Commit message: power page close
siuuuuuuuuuuuu
Connections:
- net at L1001.1: no longer U1001.9 (OUTP)
- net at C1005.1, J1001.1 (Pin_1): no longer L1001.2
- net at C1004.1, J1001.2 (Pin_2): no longer L1002.2
- net at U1001.10 (OUTN): no longer L1002.1
Other:
- moved on the sheet: L1001, L1002
Changed lines of the file:
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@@
 	(title_block
 		(title "Sensors and Audio")
-		(date "2024-12-11")
+		(date "2024-12-18")
 		(rev "1.0")
 		(company "kode.")
@@
 		(dnp no)
 		(fields_autoplaced yes)
-		(property "Reference" "#PWR01017"
+		(property "Reference" "#PWR1017"
 			(at 172.72 135.89 0)
 			(effects
@@
 			(project "cyberman"
 				(path "/0650c7a8-acba-429c-9f8e-eec0baf0bc1c/fede4c36-00cc-4d3d-b71c-5243ba232202/9419fab5-4e10-47ff-8d9d-48b1a5bf36df"
-					(reference "#PWR01017")
+					(reference "#PWR1017")
 					(unit 1)
 				)
@@
 		(dnp no)
 		(fields_autoplaced yes)
-		(property "Reference" "#PWR01013"
+		(property "Reference" "#PWR1013"
 			(at 38.1 120.65 0)
 			(effects
@@
 			(project "cyberman"
 				(path "/0650c7a8-acba-429c-9f8e-eec0baf0bc1c/fede4c36-00cc-4d3d-b71c-5243ba232202/9419fab5-4e10-47ff-8d9d-48b1a5bf36df"
-					(reference "#PWR01013")
+					(reference "#PWR1013")
 					(unit 1)
 				)
@@
 		(dnp no)
 		(fields_autoplaced yes)
-		(property "Reference" "#PWR01004"
+		(property "Reference" "#PWR1004"
 			(at 212.09 66.04 0)
 			(effects
@@
 			(project "cyberman"
 				(path "/0650c7a8-acba-429c-9f8e-eec0baf0bc1c/fede4c36-00cc-4d3d-b71c-5243ba232202/9419fab5-4e10-47ff-8d9d-48b1a5bf36df"
-					(reference "#PWR01004")
+					(reference "#PWR1004")
 					(unit 1)
 				)
@@
 		(dnp no)
 		(fields_autoplaced yes)
-		(property "Reference" "#PWR01016"
+		(property "Reference" "#PWR1016"
 			(at 160.02 135.89 0)
 			(effects
@@
 			(project "cyberman"
 				(path "/0650c7a8-acba-429c-9f8e-eec0baf0bc1c/fede4c36-00cc-4d3d-b71c-5243ba232202/9419fab5-4e10-47ff-8d9d-48b1a5bf36df"
-					(reference "#PWR01016")
+					(reference "#PWR1016")
 					(unit 1)
 				)
@@
 		(dnp no)
 		(fields_autoplaced yes)
-		(property "Reference" "#PWR01019"
+		(property "Reference" "#PWR1019"
 			(at 38.1 137.16 0)
 			(effects
@@
 			(project "cyberman"
 				(path "/0650c7a8-acba-429c-9f8e-eec0baf0bc1c/fede4c36-00cc-4d3d-b71c-5243ba232202/9419fab5-4e10-47ff-8d9d-48b1a5bf36df"
-					(reference "#PWR01019")
+					(reference "#PWR1019")
 					(unit 1)
 				)
@@
 		(dnp no)
 		(fields_autoplaced yes)
-		(property "Reference" "#PWR01011"
+		(property "Reference" "#PWR1011"
 			(at 66.04 82.55 0)
 			(effects
@@
 			(project "cyberman"
 				(path "/0650c7a8-acba-429c-9f8e-eec0baf0bc1c/fede4c36-00cc-4d3d-b71c-5243ba232202/9419fab5-4e10-47ff-8d9d-48b1a5bf36df"
-					(reference "#PWR01011")
+					(reference "#PWR1011")
 					(unit 1)
 				)
@@
 		(on_board yes)
 		(dnp no)
-		(property "Reference" "#PWR01023"
+		(property "Reference" "#PWR1023"
 			(at 248.92 148.59 0)
 			(effects
@@
 			(project "cyberman"
 				(path "/0650c7a8-acba-429c-9f8e-eec0baf0bc1c/fede4c36-00cc-4d3d-b71c-5243ba232202/9419fab5-4e10-47ff-8d9d-48b1a5bf36df"
-					(reference "#PWR01023")
+					(reference "#PWR1023")
 					(unit 1)
 				)
@@
 		(dnp no)
 		(fields_autoplaced yes)
-		(property "Reference" "#PWR01020"
+		(property "Reference" "#PWR1020"
 			(at 50.8 137.16 0)
 			(effects
@@
 			(project "cyberman"
 				(path "/0650c7a8-acba-429c-9f8e-eec0baf0bc1c/fede4c36-00cc-4d3d-b71c-5243ba232202/9419fab5-4e10-47ff-8d9d-48b1a5bf36df"
-					(reference "#PWR01020")
+					(reference "#PWR1020")
 					(unit 1)
 				)
@@
 		(on_board yes)
 		(dnp no)
-		(property "Reference" "#PWR01007"
+		(property "Reference" "#PWR1007"
 			(at 201.93 68.58 0)
 			(effects
@@
 			(project "cyberman"
 				(path "/0650c7a8-acba-429c-9f8e-eec0baf0bc1c/fede4c36-00cc-4d3d-b71c-5243ba232202/9419fab5-4e10-47ff-8d9d-48b1a5bf36df"
-					(reference "#PWR01007")
+					(reference "#PWR1007")
 					(unit 1)
 				)
@@
 		(dnp no)
 		(fields_autoplaced yes)
-		(property "Reference" "#PWR01012"
+		(property "Reference" "#PWR1012"
 			(at 160.02 119.38 0)
 			(effects
@@
 			(project "cyberman"
 				(path "/0650c7a8-acba-429c-9f8e-eec0baf0bc1c/fede4c36-00cc-4d3d-b71c-5243ba232202/9419fab5-4e10-47ff-8d9d-48b1a5bf36df"
-					(reference "#PWR01012")
+					(reference "#PWR1012")
 					(unit 1)
 				)
@@
 	)
 	(symbol
-		(lib_name "CC0402KRX7R8BB104_1")
 		(lib_id "0_capacitor_smd:CC0402KRX7R8BB104")
 		(at 201.93 55.88 0)
@@
 		(dnp no)
 		(fields_autoplaced yes)
-		(property "Reference" "#PWR01006"
+		(property "Reference" "#PWR1006"
 			(at 48.26 67.31 0)
 			(effects
@@
 			(project "cyberman"
 				(path "/0650c7a8-acba-429c-9f8e-eec0baf0bc1c/fede4c36-00cc-4d3d-b71c-5243ba232202/9419fab5-4e10-47ff-8d9d-48b1a5bf36df"
-					(reference "#PWR01006")
+					(reference "#PWR1006")
 					(unit 1)
 				)
@@
 	)
 	(symbol
-		(lib_name "CC0402KRX7R8BB104_2")
 		(lib_id "0_capacitor_smd:CC0402KRX7R8BB104")
 		(at 48.26 54.61 0)
@@
 		(dnp no)
 		(fields_autoplaced yes)
-		(property "Reference" "#PWR01009"
+		(property "Reference" "#PWR1009"
 			(at 142.24 69.85 0)
 			(effects
@@
 			(project "cyberman"
 				(path "/0650c7a8-acba-429c-9f8e-eec0baf0bc1c/fede4c36-00cc-4d3d-b71c-5243ba232202/9419fab5-4e10-47ff-8d9d-48b1a5bf36df"
-					(reference "#PWR01009")
+					(reference "#PWR1009")
 					(unit 1)
 				)
@@
 		(dnp no)
 		(fields_autoplaced yes)
-		(property "Reference" "#PWR01018"
+		(property "Reference" "#PWR1018"
 			(at 185.42 135.89 0)
 			(effects
@@
 			(project "cyberman"
 				(path "/0650c7a8-acba-429c-9f8e-eec0baf0bc1c/fede4c36-00cc-4d3d-b71c-5243ba232202/9419fab5-4e10-47ff-8d9d-48b1a5bf36df"
-					(reference "#PWR01018")
+					(reference "#PWR1018")
 					(unit 1)
 				)
@@
 	)
 	(symbol
-		(lib_name "CC0402MRX5R6BB106_1")
 		(lib_id "0_capacitor_smd:CC0402MRX5R6BB106")
 		(at 35.56 54.61 0)
@@
 		(dnp no)
 		(fields_autoplaced yes)
-		(property "Reference" "#PWR01010"
+		(property "Reference" "#PWR1010"
 			(at 250.19 73.66 0)
 			(effects
@@
 			(project "cyberman"
 				(path "/0650c7a8-acba-429c-9f8e-eec0baf0bc1c/fede4c36-00cc-4d3d-b71c-5243ba232202/9419fab5-4e10-47ff-8d9d-48b1a5bf36df"
-					(reference "#PWR01010")
+					(reference "#PWR1010")
 					(unit 1)
 				)
@@
 		(dnp no)
 		(fields_autoplaced yes)
-		(property "Reference" "#PWR01008"
+		(property "Reference" "#PWR1008"
 			(at 130.81 69.85 0)
 			(effects
@@
 			(project "cyberman"
 				(path "/0650c7a8-acba-429c-9f8e-eec0baf0bc1c/fede4c36-00cc-4d3d-b71c-5243ba232202/9419fab5-4e10-47ff-8d9d-48b1a5bf36df"
-					(reference "#PWR01008")
+					(reference "#PWR1008")
 					(unit 1)
 				)
@@
 		(dnp no)
 		(fields_autoplaced yes)
-		(property "Reference" "#PWR01005"
+		(property "Reference" "#PWR1005"
 			(at 35.56 67.31 0)
 			(effects
@@
 			(project "cyberman"
 				(path "/0650c7a8-acba-429c-9f8e-eec0baf0bc1c/fede4c36-00cc-4d3d-b71c-5243ba232202/9419fab5-4e10-47ff-8d9d-48b1a5bf36df"
-					(reference "#PWR01005")
+					(reference "#PWR1005")
 					(unit 1)
 				)
@@
 		(dnp no)
 		(fields_autoplaced yes)
-		(property "Reference" "#PWR01014"
+		(property "Reference" "#PWR1014"
 			(at 261.62 127 0)
 			(effects
@@
 			(project "cyberman"
 				(path "/0650c7a8-acba-429c-9f8e-eec0baf0bc1c/fede4c36-00cc-4d3d-b71c-5243ba232202/9419fab5-4e10-47ff-8d9d-48b1a5bf36df"
-					(reference "#PWR01014")
+					(reference "#PWR1014")
 					(unit 1)
 				)
@@
 		(dnp no)
 		(fields_autoplaced yes)
-		(property "Reference" "#PWR01022"
+		(property "Reference" "#PWR1022"
 			(at 195.58 144.78 0)
 			(effects
@@
 			(project "cyberman"
 				(path "/0650c7a8-acba-429c-9f8e-eec0baf0bc1c/fede4c36-00cc-4d3d-b71c-5243ba232202/9419fab5-4e10-47ff-8d9d-48b1a5bf36df"
-					(reference "#PWR01022")
+					(reference "#PWR1022")
 					(unit 1)
 				)
@@
 		(dnp no)
 		(fields_autoplaced yes)
-		(property "Reference" "#PWR01003"
+		(property "Reference" "#PWR1003"
 			(at 153.67 64.77 0)
 			(effects
@@
 			(project "cyberman"
 				(path "/0650c7a8-acba-429c-9f8e-eec0baf0bc1c/fede4c36-00cc-4d3d-b71c-5243ba232202/9419fab5-4e10-47ff-8d9d-48b1a5bf36df"
-					(reference "#PWR01003")
+					(reference "#PWR1003")
 					(unit 1)
 				)
@@
 		(on_board yes)
 		(dnp no)
-		(property "Reference" "#PWR01021"
+		(property "Reference" "#PWR1021"
 			(at 68.58 138.43 0)
 			(effects
@@
 			(project "cyberman"
 				(path "/0650c7a8-acba-429c-9f8e-eec0baf0bc1c/fede4c36-00cc-4d3d-b71c-5243ba232202/9419fab5-4e10-47ff-8d9d-48b1a5bf36df"
-					(reference "#PWR01021")
+					(reference "#PWR1021")
 					(unit 1)
 				)
@@
 		(dnp no)
 		(fields_autoplaced yes)
-		(property "Reference" "#PWR01002"
+		(property "Reference" "#PWR1002"
 			(at 201.93 50.8 0)
 			(effects
@@
 			(project "cyberman"
 				(path "/0650c7a8-acba-429c-9f8e-eec0baf0bc1c/fede4c36-00cc-4d3d-b71c-5243ba232202/9419fab5-4e10-47ff-8d9d-48b1a5bf36df"
-					(reference "#PWR01002")
+					(reference "#PWR1002")
 					(unit 1)
 				)
@@
 		(dnp no)
 		(fields_autoplaced yes)
-		(property "Reference" "#PWR01024"
+		(property "Reference" "#PWR1024"
 			(at 73.66 151.13 0)
 			(effects
@@
 			(project "cyberman"
 				(path "/0650c7a8-acba-429c-9f8e-eec0baf0bc1c/fede4c36-00cc-4d3d-b71c-5243ba232202/9419fab5-4e10-47ff-8d9d-48b1a5bf36df"
-					(reference "#PWR01024")
+					(reference "#PWR1024")
 					(unit 1)
 				)
@@
 		(on_board yes)
 		(dnp no)
-		(property "Reference" "#PWR01015"
+		(property "Reference" "#PWR1015"
 			(at 124.46 130.81 0)
 			(effects
@@
 			(project "cyberman"
 				(path "/0650c7a8-acba-429c-9f8e-eec0baf0bc1c/fede4c36-00cc-4d3d-b71c-5243ba232202/9419fab5-4e10-47ff-8d9d-48b1a5bf36df"
-					(reference "#PWR01015")
+					(reference "#PWR1015")
 					(unit 1)
 				)
@@
 		(dnp no)
 		(fields_autoplaced yes)
-		(property "Reference" "#PWR01001"
+		(property "Reference" "#PWR1001"
 			(at 35.56 49.53 0)
 			(effects
@@
 			(project "cyberman"
 				(path "/0650c7a8-acba-429c-9f8e-eec0baf0bc1c/fede4c36-00cc-4d3d-b71c-5243ba232202/9419fab5-4e10-47ff-8d9d-48b1a5bf36df"
-					(reference "#PWR01001")
+					(reference "#PWR1001")
 					(unit 1)
 				)
